Commit message: NOT WORKING - Cartpole Spawns in Gazebo

File: src/cartpole/urdf/xacro/cartpole_gazebo_urdf.urdf.xacro (robot description, xacro)
@@ -50,5 +50,5 @@
         <box size="0.05 0.05 1.0"/>
       </geometry>
-      <origin rpy="0 0 0" xyz="0 0 0.5"/>
+      <origin rpy="0 0 0" xyz="0 0 -0.5"/>
       <material name="white">
         <color rgba="1 1 1 1"/>
@@ -57,5 +57,5 @@
     <inertial>
     <origin xyz="0 0 0.5"/>
-      <mass value="10"/>
+      <mass value="2"/>
       <inertia ixx="1.0" ixy="0.0" ixz="0.0" iyy="1.0" iyz="0.0" izz="1.0"/>
     </inertial>
@@ -78,15 +78,24 @@
     </actuator>
   </transmission>
+  <ros2_control name="GazeboSystem" type="system">
+    <hardware>
+      <plugin>gazebo_ros2_control/GazeboSystem</plugin>
+    </hardware>
+    <joint name="slider_to_cart">
+      <command_interface name="effort">
+        <param name="min">-1000</param>
+        <param name="max">1000</param>
+      </command_interface>
+      <state_interface name="position">
+        <param name="initial_value">1.0</param>
+      </state_interface>
+      <state_interface name="velocity"/>
+      <state_interface name="effort"/>
+    </joint>
+  </ros2_control>
   <gazebo>
-	<plugin name="gazebo_ros_control" filename="libgazebo_ros_control.so">
-		<robotNamespace>/</robotNamespace>
-		<robotSimType>gazebo_ros_control/DefaultRobotHWSim</robotSimType>
-	</plugin>
-	<plugin name="joint_state_publisher" filename="libgazebo_ros_joint_state_publisher.so">
-		<robotNamespace>/cart_pole</robotNamespace>
-		<jointName>cart_to_pole, slider_to_cart</jointName>
-		<updateRate>100</updateRate>
-		<alwaysOn>true</alwaysOn>
-	</plugin>
+    <plugin filename="libgazebo_ros2_control.so" name="gazebo_ros2_control">
+      <parameters>$(find cartpole)/config/cartpole_controller.yaml</parameters>
+    </plugin>
   </gazebo>
 </robot>
