Commit message: Working cartpole controller in gazebo

File: src/cartpole/urdf/xacro/cartpole_urdf.urdf.xacro (robot description, xacro)
@@ -78,23 +78,25 @@
     </actuator>
   </transmission>
-  <ros2_control name="GazeboSystem" type="system">
-    <hardware>
-      <plugin>gazebo_ros2_control/GazeboSystem</plugin>
-    </hardware>
-    <joint name="slider_to_cart">
-      <command_interface name="effort">
-        <param name="min">-1000</param>
-        <param name="max">1000</param>
-      </command_interface>
-      <state_interface name="position">
-        <param name="initial_value">1.0</param>
-      </state_interface>
-      <state_interface name="velocity"/>
-      <state_interface name="effort"/>
-    </joint>
-  </ros2_control>
   <gazebo>
-    <plugin filename="libgazebo_ros2_control.so" name="gazebo_ros2_control">
-      <parameters>$(find cartpole)/config/cart_pole_controller.yaml</parameters>
+    <plugin
+      filename="libignition-gazebo-joint-controller-system.so"
+      name="ignition::gazebo::systems::JointController">
+      <joint_name>cart_to_pole</joint_name>
+      <use_force_commands>true</use_force_commands>
+      <topic>/cartpole/cmd</topic>
+      <initial_velocity>0.0</initial_velocity>
+      <p_gain>100.0</p_gain>
+      <i_gain>0.01</i_gain>
+      <d_gain>10.0</d_gain>
+    </plugin>
+    <plugin
+      filename="libignition-gazebo-joint-state-publisher-system.so"
+      name="ignition::gazebo::systems::JointStatePublisher">
+      <joint_name>cart_to_pole</joint_name>
+    </plugin>
+    <plugin
+      filename="libignition-gazebo-joint-state-publisher-system.so"
+      name="ignition::gazebo::systems::JointStatePublisher">
+      <joint_name>slider_to_cart</joint_name>
     </plugin>
   </gazebo>

Commit message: Moving variables to yaml config

File: src/cartpole/urdf/xacro/cartpole_urdf.urdf.xacro (robot description, xacro)
@@ -1,4 +1,14 @@
 <?xml version="1.0"?>
 <robot name="cartpole" xmlns:xacro="http://ros.org/wiki/xacro">
+  <xacro:property name="cartpole_params" value="$(find cartpole)/config/cartpole_params.yaml" />
+  <xacro:property name="load_params" value="${xacro.load_yaml(cartpole_params)}" />
+  <xacro:property name="params" value="${load_params['cartpole_parameters']['ros__parameters']}" />
+  <xacro:property name="cart_mass"  value="${params['cart_mass']}" />
+  <xacro:property name="pole_mass"  value="${params['pole_mass']}" />
+  <xacro:property name="pole_len"  value="${params['pole_len']}" />
+  <xacro:property name="pole_org"  value="${params['pole_org']}" />
+  <xacro:property name="prop_gain"  value="${params['prop_gain']}" />
+  <xacro:property name="int_gain"  value="${params['int_gain']}" />
+  <xacro:property name="diff_gain"  value="${params['diff_gain']}" />
   <link name="world"/>
   <link name="slideBar">
@@ -28,5 +38,5 @@
     </visual>
     <inertial>
-      <mass value="1"/>
+      <mass value="${cart_mass}"/>
       <inertia ixx="1.0" ixy="0.0" ixz="0.0" iyy="1.0" iyz="0.0" izz="1.0"/>
     </inertial>
@@ -48,7 +58,7 @@
     <visual>
       <geometry>
-        <box size="0.05 0.05 1.0"/>
+        <box size="0.05 0.05 ${pole_len}"/>
       </geometry>
-      <origin rpy="0 0 0" xyz="0 0 -0.5"/>
+      <origin rpy="0 0 0" xyz="0 0 ${pole_org}"/>
       <material name="white">
         <color rgba="1 1 1 1"/>
@@ -57,5 +67,5 @@
     <inertial>
     <origin xyz="0 0 0.5"/>
-      <mass value="2"/>
+      <mass value="${pole_mass}"/>
       <inertia ixx="1.0" ixy="0.0" ixz="0.0" iyy="1.0" iyz="0.0" izz="1.0"/>
     </inertial>
@@ -86,7 +96,7 @@
       <topic>/cartpole/cmd</topic>
       <initial_velocity>0.0</initial_velocity>
-      <p_gain>100.0</p_gain>
-      <i_gain>0.01</i_gain>
-      <d_gain>10.0</d_gain>
+      <p_gain>${prop_gain}</p_gain>
+      <i_gain>${int_gain}</i_gain>
+      <d_gain>${diff_gain}</d_gain>
     </plugin>
     <plugin

Commit message: Fixed physics issue with cartpole

File: src/cartpole/urdf/xacro/cartpole_urdf.urdf.xacro (robot description, xacro)
@@ -66,5 +66,5 @@
     </visual>
     <inertial>
-    <origin xyz="0 0 0.5"/>
+    <origin xyz="0 0 ${pole_org}"/>
       <mass value="${pole_mass}"/>
       <inertia ixx="1.0" ixy="0.0" ixz="0.0" iyy="1.0" iyz="0.0" izz="1.0"/>
